File: Power-distribution-board/Power-distribution-board.kicad_sch (KiCad schematic)
At the start: 22 parts, among them U3 TPS62933

Commit message: Add files via upload
Parts:
- added JP2: Jumper_3_Bridged12, symbol Jumper:Jumper_3_Bridged12
- added U4, U5, U6, U7, U8, U9: ~, symbol Power_distribution:WAGO2T
Connections:
- net GND: now also JP2.1 (A)
- net at C1.1, C2.1, C3.1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: now also U4.1, U5.1, U6.1, U7.1, U8.1, U9.1
- net at R1.2, R2.1: now also JP2.2 (C)
- net at U2.1: now also Aux.1 (+)
- net at U2.2: now also Aux.2 (-)
- net at U3.2 (EN): now also JP2.3 (B)
- new net: U1.2, U4.2, U5.2, U6.2, U7.2, U8.2, U9.2
- new net Motor 1 +: U4.1
- new net Motor 1 -: U4.2
- new net Motor 2 +: U5.1
- new net Motor 2 -: U5.2
- new net Motor 3 +: U6.1
- new net Motor 3 -: U6.2
- new net Motor 4 +: U7.1
- new net Motor 4 -: U7.2
- new net Motor 5 +: U8.1
- new net Motor 5 -: U8.2
- new net Motor 6 +: U9.1
- new net Motor 6 -: U9.2
Other:
- note added: "WAGO 10AWG Output"
- moved on the sheet: Aux, C1, C2, C3, C4, C5, C6, C7, C8, JP1, L1, R1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
