File: Power-distribution-board.kicad_sch (KiCad schematic)
At the start: 104 parts, among them J1 MRCBP-V-40A, J10 2606-1104/020-000, J11 Conn_01x02_Pin, J12 2606-1104/020-000, J13 2606-1104/020-000, J14 2606-1104/020-000, J15 2606-1104/020-000, J16 2606-1104/020-000, J2 MRCBP-V-40A, J3 MRCBP-V-40A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

Commit message: Updated connectors and started resistor values
Parts:
- removed C2: C, symbol Device:C
- removed J14: 2606-1104/020-000, CONN4_2606-1104/020-000_WAG, symbol wago:2606-1104_020-000
- removed R1, R2, R4: R, symbol Device:R
- C11: value C -> 0.1
- R10, R14, R24, R27, R30, R33: value R -> 0.01
- R8, R9: value R -> 10
Connections:
- net JETSON+ is gone; now on net MOT4: J16.3
- net AUX+: now also J12.1
- net BAT-: now also J10.2, J10.4, J16.2, J16.4; no longer J15.1, J15.3
- net MOT1: now also R11.2
- net MOT2: now also J10.3, R15.2; no longer J10.2
- net MOT3: now also J16.1, R16.2; no longer J10.3
- net MOT4: now also R19.2; no longer J10.4
- net MOT5: now also J15.1, R20.2; no longer J16.1
- net MOT6: now also J15.3, R21.2; no longer J16.2
- net AUX-: now reaches J12.2
- net AUX-: now also J13.1; no longer R15.2
- net at J12.4: no longer R19.2
- net at J12.3: no longer R16.2
- removed net JETSON-: J13.1, J16.4
- no-connect marks 52 -> 56
Other:
- moved on the sheet: J15

Commit message: Update INA220 circuit
Parts:
- C1: value C -> 0.1uF
Connections:
- net BAT- is gone; now on net GND: J10.2, J10.4, J13.3, J15.2, J15.4, J16.2, J16.4
- net 5VOUT: no longer C29.1, C30.1, C31.1, L2.2, R40.1
- net AUX-: now also C1.2, U3.7 (GND)
- net GND: no longer C1.2, U3.7 (GND)
- net 3.3V TO 5V renamed 5V
- net 5V: now also C29.1, C30.1, C31.1, L2.2, R40.1
Other:
- note added: "I2C Address: 0x40"
- note added: "I2C Address: 0x46"
- note added: "Use Aux- as GND since VBus (aux battery voltage) is measured with reference to GND of INA220"
- moved on the sheet: R10

Commit message: Update Power-distribution-board.kicad_sch
Parts:
- removed R11, R15, R16, R19, R20, R21: R, symbol Device:R
Connections:
- net MOT1 is gone; now on net IC1: J10.1, R10.1, R9.1
- net MOT2 is gone; now on net IC2: J10.3, R13.1, R14.1
- net MOT3 is gone; now on net IC3: J16.1, R23.1, R24.1
- net MOT4 is gone; now on net IC4: J16.3, R26.1, R27.1
- net MOT5 is gone; now on net IC5: J15.1, R29.1, R30.1
- net MOT6 is gone; now on net IC6: J15.3, R32.1, R33.1

Commit message: changed 15-5v buck converter and fix current sensors
Parts:
- removed 15-5VRM1: TPS62933DRLR, TPS62933DRLR:SOTFL50P160X60-8N, symbol powerdist:TPS62933DRLR
- removed C24, C25: 10uF, symbol Device:C
- removed C26, C28, C31: 100nF, symbol Device:C
- removed C27: 33nF, symbol Device:C
- removed C29, C30: 22uF, symbol Device:C
- removed J11: Conn_01x02_Pin, symbol Connector:Conn_01x02_Pin
- removed J8: Conn_01x03_Pin, symbol Connector:Conn_01x03_Pin
- removed L2: 6.8uH, symbol Device:L
- removed R34: 511k, symbol Device:R
- removed R35: 88.7k, symbol Device:R
- removed R36, R38: 0, symbol Device:R
- removed R37: 10.2k, symbol Device:R
- removed R39: 53.55k, symbol Device:R
- removed R40: 49.9, symbol Device:R
- added C2: 0.1 uF, symbol Device:C
- added C32: 1.0 uF, symbol Device:C
- added R1: 240 ohm, symbol Device:R
- added R2: 715 ohm, symbol Device:R
- added U4: LM317_SOT-223, Package_TO_SOT_SMD:SOT-223-3_TabPin2, symbol Regulator_Linear:LM317_SOT-223
Connections:
- net 15VIN: now also C2.1, U4.3 (VI)
- net 5VOUT: now also C32.1, R1.1, U4.2 (VO)
- net GND: now also C2.2, C32.2, R2.2
- net IC1 renamed MOT1
- net MOT1: no longer U12.8 (VBUS)
- net IC2 renamed MOT2
- net MOT2: no longer U13.8 (VBUS)
- net IC3 renamed MOT3
- net MOT3: no longer U14.8 (VBUS)
- net IC4 renamed MOT4
- net MOT4: no longer U15.8 (VBUS)
- net IC5 renamed MOT5
- net MOT5: no longer U16.8 (VBUS)
- net IC6 renamed MOT6
- net MOT6: no longer U17.8 (VBUS)
- new net: R1.2, R2.1, U4.1 (ADJ)
- no-connect marks 56 -> 62
Other:
- note added: "15-5v buck converter"
- note added: "5 to 3.3 V buck converter"
- note removed: "15V-5V Buck Converter"
- note removed: "from BATTERY"
- note removed: "to ESP"
