File: Power-distribution-board.kicad_sch (KiCad schematic)
At the start: 89 parts, among them J1 178.6165.0001 breaker, J10 2606-1104/020-000, J12 2606-1104/020-000, J13 2606-1104/020-000, J15 2606-1104/020-000, J16 2606-1104/020-000, J2 178.6165.0001 breaker, J3 178.6165.0001 breaker, J4 178.6165.0001 breaker, J5 178.6165.0001 breaker, J6 178.6165.0001 breaker, J7 Screw_Terminal_01x03, J9 USB_C_Receptacle_USB2.0_14P, SW1 SW_Nidec_CAS-120A1, U1 ESP32-S3-WROOM-1, U11 TJA1051TK-3, U12 INA220BIDGSR, U13 INA220BIDGSR, U14 INA220BIDGSR, U15 INA220BIDGSR, U16 INA220BIDGSR, U17 INA220BIDGSR, U18 CP2102N-Axx-xQFN24, U2 LM3940IT-3.3, U3 INA220BIDGSR, U4 LM317_SOT-223, U5 TM1637, U6 CC56-12EWA

Commit message: traces done
has some error and warnings tho
Connections:
- net BAT+ is gone; now on net BATP: J1.2 (Pin_2), J13.4, J2.2 (Pin_2), J3.2 (Pin_2), J4.2 (Pin_2), J5.2 (Pin_2), J6.2 (Pin_2), R10.2, R12.2, R14.2, R22.2, R24.2, R25.2, R27.2, R28.2, R30.2, R31.2, R33.2, R8.2
- net 15VIN renamed BATP
Changed lines of the file:
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@@
 		)
 	)
-	(label "15VIN"
+	(label "BATP"
 		(at 267.97 194.31 180)
 		(effects
@@
 		)
 	)
-	(label "BAT+"
+	(label "BATP"
 		(at 212.09 302.26 0)
 		(effects
@@
 		)
 	)
-	(label "BAT+"
+	(label "BATP"
 		(at 115.57 299.72 0)
 		(effects
@@
 		)
 	)
-	(label "BAT+"
+	(label "BATP"
 		(at 214.63 209.55 0)
 		(effects
@@
 		)
 	)
-	(label "BAT+"
+	(label "BATP"
 		(at 114.3 255.27 0)
 		(effects
@@
 		)
 	)
-	(label "BAT+"
+	(label "BATP"
 		(at 90.17 63.5 0)
 		(effects
@@
 		)
 	)
-	(label "BAT+"
+	(label "BATP"
 		(at 118.11 212.09 0)
 		(effects
@@
 		)
 	)
-	(label "BAT+"
+	(label "BATP"
 		(at 213.36 256.54 0)
 		(effects
@@
 		)
 	)
-	(label "BAT+"
+	(label "BATP"
 		(at 80.01 40.64 180)
 		(effects
