File: Power-distribution-board.kicad_sch (KiCad schematic)
At the start: 100 parts, among them J1 Conn_01x03_Pin, J10 2606-1104/020-000, J11 178.6165.0001, J12 2606-1104/020-000, J13 2606-1104/020-000, J14 178.6165.0001, J15 2606-1104/020-000, J16 2606-1104/020-000, J17 178.6165.0001, J18 178.6165.0001, J19 178.6165.0001, J7 Screw_Terminal_01x03, J8 178.6165.0001, J9 USB_C_Receptacle_USB2.0_14P, U1 ESP32-S3-WROOM-1, U11 TJA1051TK-3, U12 INA220BIDGSR, U13 INA220BIDGSR, U14 INA220BIDGSR, U15 INA220BIDGSR, U16 INA220BIDGSR, U17 INA220BIDGSR, U18 CP2102N-Axx-xQFN24, U2 LM3940IT-3.3, U3 INA220BIDGSR, U5 TM1637, U6 CC56-12EWA

Commit message: updated version
-added common ground point for aux-, batn, and signal gnd
-changed usb stackup so usb is powered by LDO 3v3
-changed wago terminal for battery (rated 60A)
Parts:
- removed C3: 10µ, Capacitor_SMD:C_0402_1005Metric, symbol Device:C
- removed C4: 0.1µ, Capacitor_SMD:C_0402_1005Metric, symbol Device:C
- removed C5: 0.1uF, Capacitor_SMD:C_0402_1005Metric, symbol Device:C
- removed C6: 10µF, Capacitor_SMD:C_0402_1005Metric, symbol Device:C
- removed D2: SP0503BAHT, Package_TO_SOT_SMD:SOT-143, symbol Power_Protection:SP0503BAHT
- removed D4: D, pdb_footprints:USC_TOS, symbol Device:D
- removed J13: 2606-1104/020-000, pdb_footprints:CONN4_2606-1104&slash_020-000_WAG, symbol wago:2606-1104_020-000
- removed J9: USB_C_Receptacle_USB2.0_14P, Connector_USB:USB_C_Receptacle_HRO_TYPE-C-31-M-12, symbol Connector:USB_C_Receptacle_USB2.0_14P
- removed R45, R46: 5.1k, Resistor_SMD:R_0402_1005Metric, symbol Device:R
- removed R5: 22.1k, Resistor_SMD:R_0402_1005Metric, symbol Device:R
- removed R6: 47.5k, Resistor_SMD:R_0402_1005Metric, symbol Device:R
- removed R7: 10k, Resistor_SMD:R_0402_1005Metric, symbol Device:R
- removed U18: CP2102N-Axx-xQFN24, Package_DFN_QFN:QFN-24-1EP_4x4mm_P0.5mm_EP2.6x2.6mm, symbol Interface_USB:CP2102N-Axx-xQFN24
- added C2: 4.7u, Capacitor_SMD:C_0402_1005Metric, symbol Device:C
- added C32: 0.1u, Capacitor_SMD:C_0201_0603Metric, symbol Device:C
- added D1: SP0503BAHT, Package_TO_SOT_SMD:SOT-143, symbol Power_Protection:SP0503BAHT
- added J2: 2616-1102/020-000, CONN2_2616-1102/020-000_WAG, symbol Wago 60A:2616-1102_020-000
- added J3: USB_C_Receptacle_USB2.0_14P, Connector_USB:USB_C_Receptacle_HRO_TYPE-C-31-M-12, symbol Connector:USB_C_Receptacle_USB2.0_14P
- added NT1: NetTie_3_Tee, NetTie:NetTie-3_THT_Pad1.0mm, symbol Device:NetTie_3_Tee
- added R1, R2: 4.7k, Resistor_SMD:R_0402_1005Metric, symbol Device:R
- added R16: 1k, Resistor_SMD:R_0402_1005Metric, symbol Device:R
- added R35: 22.1k, Resistor_SMD:R_0402_1005Metric, symbol Device:R
- added R36: 47.5k, Resistor_SMD:R_0402_1005Metric, symbol Device:R
- added R37, R38: 5.1k, Resistor_SMD:R_0402_1005Metric, symbol Device:R
- added U4: CP2102N-Axx-xQFN24, Package_DFN_QFN:QFN-24-1EP_4x4mm_P0.5mm_EP2.6x2.6mm, symbol Interface_USB:CP2102N-Axx-xQFN24
- R20: value 0 -> 0.3
- R21: footprint Resistor_SMD:R_0805_2012Metric -> Resistor_SMD:R_01005_0402Metric
Connections:
- net 3.3V: now also C1.1, C14.1, C15.1, C16.1, C18.1, C20.1, C22.1, U12.6 (VS), U13.2 (A0), U13.6 (VS), U14.6 (VS), U15.6 (VS), U16.1 (A1), U16.6 (VS), U17.1 (A1), U17.2 (A0), U17.6 (VS), U3.1 (A1), U3.6 (VS), C2.2, C32.2, R1.1, R16.1, R2.1, U4.5 (VIO), U4.6 (VDD), U4.7 (VREGIN)
- net 5V: no longer C1.1, C14.1, C15.1, C16.1, C18.1, C20.1, C22.1, U12.6 (VS), U13.2 (A0), U13.6 (VS), U14.6 (VS), U15.6 (VS), U16.1 (A1), U16.6 (VS), U17.1 (A1), U17.2 (A0), U17.6 (VS), U3.1 (A1), U3.6 (VS)
- net AUX+: now also J12.3
- net AUX-: now also J12.4, NT1.2
- net BATN: now also J2.4 (2_1), NT1.1
- net BATP: now also J2.1 (1_1)
- net CLK: now also C27.2, R3.2, U5.18 (CLK)
- net DIO: now also C28.1, R4.2, U5.17 (DIO)
- net GND: now also C2.1, C32.1, D1.1 (A), J3.A1 (GND), J3.A12 (GND), J3.B1 (GND), J3.B12 (GND), J3.S1 (SHIELD), NT1.3, R36.2, R37.2, R38.2, U4.2 (GND), U4.25 (GND)
- net MOT1: no longer J10.1
- net MOT1_OUT: now also J10.1
- net MOT2: no longer J10.3
- net MOT2_OUT: now also J10.3
- net MOT3: no longer J16.1
- net MOT3_OUT: now also J16.1
- net MOT4: no longer J16.3
- net MOT4_OUT: now also J16.3
- net MOT5: no longer J15.1
- net MOT5_OUT: now also J15.1
- net MOT6: no longer J15.3
- net MOT6_OUT: now also J15.3
- net SCL: now also R2.2
- net SDA: now also R1.2
- net UART RX: now also U4.21 (TXD)
- net UART TX: now also U4.20 (RXD)
- net at 15-5VRM1.8 (FB), R19.2, R21.2: no longer R21.1, R34.2
- new net: R35.2, R36.1
- new net: D1.2 (K), J3.A4 (VBUS), J3.A9 (VBUS), J3.B4 (VBUS), J3.B9 (VBUS), R35.1, U4.8 (VBUS)
- new net: D1.3 (K), J3.A7 (D-), J3.B7 (D-), U4.4 (D-)
- new net: D1.4 (K), J3.A6 (D+), J3.B6 (D+), U4.3 (D+)
- new net: R21.1, R34.2
- new net: R16.2, U4.9 (~{RST})
- new net CC1: J3.A5 (CC1), R37.1
- new net CC2: J3.B5 (CC2), R38.1
- no-connect marks 64 -> 61
Other:
- note added: "Pull up resistors"
- note added: "bypass capacitors - place close to vdd pin"
- note added: "common ground point, place near BATN (J2)"
- moved on the sheet: 15-5VRM1, C11, C12, C14, C15, C16, C17, C18, C19, C20, C21, C22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

Commit message: much progress has been made
layout is complete. looks very geometrlic. : -D
Parts:
- added C3, C4, C5, C6: 0.1u, Capacitor_SMD:C_0201_0603Metric, symbol Device:C
- added J4, J5: 178.6165.0001, PDB Footprint Library:CONN_178.6165.0001_LTF, symbol PDB_symbols:178.6165.0001
- added J6: 2606-1104/020-000, PDB Footprint Library:CONN4_2606-1104&slash_020-000_WAG, symbol wago:2606-1104_020-000
- added R39, R40, R5, R6: 0, Resistor_SMD:R_0805_2012Metric, symbol Device:R
- added R41, R7: 1m, PDB Footprint Library:RES_3920R_1L00x_BRN-M, symbol Device:R
- added U7, U8: INA220BIDGSR, PDB Footprint Library:DGS10, symbol INA220:INA220BIDGSR
- C1, C11, C12, C14, C15, C16, C17, C18, C19, C20, C21, C22, C23: footprint Capacitor_SMD:C_0805_2012Metric -> Capacitor_SMD:C_0201_0603Metric
- C10, C13, C2, C9: footprint Capacitor_SMD:C_0402_1005Metric -> Capacitor_SMD:C_0805_2012Metric
- J10, J12, J15, J16: footprint pdb_footprints:CONN4_2606-1104&slash_020-000_WAG -> PDB Footprint Library:CONN4_2606-1104&slash_020-000_WAG
- J2: footprint CONN2_2616-1102/020-000_WAG -> PDB Footprint Library:CONN2_2616-1102&slash_020-000_WAG
- R21: footprint Resistor_SMD:R_01005_0402Metric -> Resistor_SMD:R_0805_2012Metric
- U12, U13, U14, U15, U16, U17, U3: footprint pdb_footprints:DGS10 -> PDB Footprint Library:DGS10
Connections:
- net 3.3V: now also C3.1, C5.1, U7.1 (A1), U7.6 (VS), U8.1 (A1), U8.6 (VS)
- net BATN: now also J6.2, J6.4
- net BATP: now also J4.1, J5.1
- net GND: now also C3.2, C5.2, U7.7 (GND), U8.7 (GND)
- net SCL: now also U7.5 (SCL), U8.2 (A0), U8.5 (SCL)
- net SDA: now also U7.2 (A0), U7.4 (SDA), U8.4 (SDA)
- net at R35.2, R36.1: now also U4.8 (VBUS)
- net at D1.2 (K), J3.A4 (VBUS), J3.A9 (VBUS)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: no longer U4.8 (VBUS)
- new net: C4.2, R6.2, U7.9 (VIN-)
- new net: C6.2, R40.2, U8.9 (VIN-)
- new net: C4.1, R5.1, U7.10 (VIN+)
- new net: C6.1, R39.1, U8.10 (VIN+)
- new net MOT7: J4.8, R5.2, R7.2
- new net MOT7_OUT: J6.1, R6.1, R7.1
- new net MOT8: J5.8, R39.2, R41.2
- new net MOT8_OUT: J6.3, R40.1, R41.1
- no-connect marks 61 -> 65
Other:
- note added: "ESP bypass capacitors"
- note added: "I2C Address: 0x47"
- moved on the sheet: C1, C10, C13, C2, C27, C28, C29, C30, C32, C7, C8, C9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
