File: Power-distribution-board.kicad_pcb (KiCad board)
At the start: 4 copper layers, 142.3 x 104.1 mm, 90 parts, among them J1 178.6165.0001 breaker, J10 2606-1104/020-000, J12 2606-1104/020-000, J13 2606-1104/020-000, J15 2606-1104/020-000, J16 2606-1104/020-000, J2 178.6165.0001 breaker, J3 178.6165.0001 breaker, J4 178.6165.0001 breaker, J5 178.6165.0001 breaker, J6 178.6165.0001 breaker, J7 Screw_Terminal_01x03, J9 USB_C_Receptacle_USB2.0_14P, SW1 SW_Nidec_CAS-120A1, U1 ESP32-S3-WROOM-1, U11 TJA1051TK-3, U12 INA220BIDGSR, U13 INA220BIDGSR, U14 INA220BIDGSR, U15 INA220BIDGSR, U16 INA220BIDGSR, U17 INA220BIDGSR, U18 CP2102N-Axx-xQFN24, U2 LM3940IT-3.3, U3 INA220BIDGSR, U4 LM317_SOT-223, U5 TM1637, U6 CC56-12EWA

Commit message: traces done
has some error and warnings tho
Parts:
- moved C13 16.9 mm to (115.7, 75.0)
- moved C20 12.6 mm to (173.0, 94.0), turned to 180 degrees
- moved C32 2.73 mm to (156.9, 75.0), turned to 0 degrees
- moved C11 1.03 mm to (147.8, 82.0), turned to 180 degrees
- moved R2 0.54 mm to (153.9, 78.2), turned to 0 degrees
- moved U1 0.53 mm to (102.2, 64.3)
- moved C26 0.35 mm to (90.6, 60.4), turned to -90 degrees
Connections:
- C2 pad 1: /15VIN -> /BATP
- J1 pad 2: /BAT+ -> /BATP
- J13 pad 4: /BAT+ -> /BATP
- J2 pad 2: /BAT+ -> /BATP
- J3 pad 2: /BAT+ -> /BATP
- J4 pad 2: /BAT+ -> /BATP
- J5 pad 2: /BAT+ -> /BATP
- J6 pad 2: /BAT+ -> /BATP
- R10 pad 2: /BAT+ -> /BATP
- R12 pad 2: /BAT+ -> /BATP
- R14 pad 2: /BAT+ -> /BATP
- R22 pad 2: /BAT+ -> /BATP
- R24 pad 2: /BAT+ -> /BATP
- R25 pad 2: /BAT+ -> /BATP
- R27 pad 2: /BAT+ -> /BATP
- R28 pad 2: /BAT+ -> /BATP
- R30 pad 2: /BAT+ -> /BATP
- R31 pad 2: /BAT+ -> /BATP
- R33 pad 2: /BAT+ -> /BATP
- R8 pad 2: /BAT+ -> /BATP
- U4 pad 3: /15VIN -> /BATP
Routing:
- net /SCL: track 0.00 -> 173.0 mm, vias 0 -> 11
- net /SDA: track 0.00 -> 172.2 mm, vias 0 -> 11
- net GND: track 0.00 -> 151.3 mm, vias 0 -> 46
- net /AUX-: track 0.00 -> 150.7 mm, vias 0 -> 2
- net /BATP: track 0.00 -> 145.4 mm, vias 0 -> 52
- net /AUX+: track 0.00 -> 142.3 mm, vias 0 -> 3
- net /5V: track 0.00 -> 129.4 mm, vias 0 -> 38
- net /MOT5: track 0.00 -> 85.5 mm, vias 0 -> 2
- net /3.3V: track 0.00 -> 60.6 mm, vias 0 -> 7
- net Net-(D4-A): track 0.00 -> 46.8 mm, vias 0 -> 4
- net Net-(U5-GRID3): track 0.00 -> 43.3 mm, vias 0 -> 1
- net /MOT2: track 0.00 -> 42.0 mm, vias 0 -> 2
- net /MOT1: track 0.00 -> 41.5 mm, vias 0 -> 2
- net Net-(U5-GRID1): track 0.00 -> 40.5 mm, vias 0 -> 1
- net Net-(U5-GRID2): track 0.00 -> 40.5 mm, vias 0 -> 1
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- added copper zone on In2.Cu, net /BATP
- removed copper zone on In2.Cu, net /15VIN
- removed copper zone on In2.Cu, net /BAT+

Commit message: fixed design rules errors
Routing:
- net /5V: track 129.4 -> 159.0 mm, vias 38 -> 45
- net /BATP: track 145.4 -> 156.8 mm, vias 52 -> 54
- net GND: track 151.3 -> 156.7 mm, vias 46 -> 49
- net Net-(U5-SEG7/KS7): track 14.3 -> 17.5 mm, vias 1 -> 3
- net /3.3V: track 60.6 -> 61.6 mm
